File: LinTempCont_4ch_proto.brd (EAGLE design)
At the start: 330.2 x 76.2 mm, 207 parts, among them IC1 LM393D, IC10 AD5262, IC2 LM393D, IC3 AD5624R, IC4 AD5262, IC5 AD5262, IC7 LM393D, IC8 AD5262, IC9 LM393D, T1 MMBT3904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

Commit message: Schematic updates and progress routing both boards
Parts:
- removed R16, R17, R50, R51, R68, R69, R86, R87: 0, rlc-jqi:0603
- removed RI1, RI2, RI3, RP1, RP2, RP3: DNP, rlc-jqi:0603
- R35: device rlc-jqi:0805 -> rlc-jqi:0603
- moved C4 307.0 mm to (39.4, 31.8), turned to 90 degrees
- moved C5 300.1 mm to (41.9, 31.8), turned to 90 degrees
- moved C6 293.2 mm to (44.5, 31.8), turned to 90 degrees
- moved C7 286.3 mm to (47.0, 31.8), turned to 90 degrees
- moved R22 262.8 mm to (41.3, 26.0)
- moved R23 258.2 mm to (41.3, 28.6), turned to 180 degrees
- moved R24 253.0 mm to (46.4, 25.4)
- moved R25 248.4 mm to (46.4, 27.9), turned to 180 degrees
- moved R52 210.1 mm to (120.7, 17.8)
- moved R39 208.6 mm to (170.2, 26.7), turned to 180 degrees
- moved R44 206.7 mm to (157.5, 26.7)
- moved R45 205.8 mm to (153.7, 26.7)
- moved TP11 205.7 mm to (142.2, 64.8)
- moved R40 203.2 mm to (170.2, 29.2)
- moved R43 198.6 mm to (161.3, 40.6), turned to 90 degrees
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Connections:
- removed net N$18: IC4.3, IC4.4, R16.1
- removed net N$2: JP1.6, R14.1, R15.1
- removed net N$20: IC4.14, IC4.15, R17.2
- removed net N$33: IC5.3, IC5.4, R50.1
- removed net N$34: IC5.14, IC5.15, R51.2
- removed net N$48: IC8.3, IC8.4, R68.1
- removed net N$49: IC8.14, IC8.15, R69.2
- removed net N$63: IC10.3, IC10.4, R86.1
- removed net N$64: IC10.14, IC10.15, R87.2
- new net N$69: JP1.8, R14.1, R15.1
- net +1V_1: now also IC4.14, IC4.15, IC4.3, IC4.4, JP1.3; no longer JP1.11, R16.2, R17.1
- net +1V_2: now also IC5.14, IC5.15, IC5.3, IC5.4, JP2.3; no longer JP2.11, R50.2, R51.1, RI1.2, RP1.1
- net +1V_3: now also IC8.14, IC8.15, IC8.3, IC8.4, JP8.3; no longer JP8.11, R68.2, R69.1, RI2.2, RP2.1
- net +1V_4: now also IC10.14, IC10.15, IC10.3, IC10.4, JP11.3; no longer JP11.11, R86.2, R87.1, RI3.2, RP3.1
- net 2.5V: now also JP1.9, JP11.9, JP2.9, JP8.9; no longer JP1.10, JP11.10, JP2.10, JP8.10
- net ACT_T2: now also U$1.23/A9; no longer U$1.20/A6
- net ACT_T3: now also U$1.21/A7; no longer U$1.18/A4
- net ACT_T4: now also U$1.19/A5; no longer U$1.16/A2
- net AGND: now also JP1.12, JP11.12, JP2.12, JP8.12; no longer JP1.2, JP11.2, JP2.2, JP8.2
- net CS_DAC: now also U$1.6; no longer U$1.14/A0
- net CS_LCD: now also U$1.12; no longer U$1.5
- net CS_POT1: now also U$1.2; no longer U$1.8
- net CS_POT2: now also U$1.3; no longer U$1.9
- net CS_POT3: now also U$1.4; no longer U$1.10
- net CS_POT4: now also U$1.5; no longer U$1.12
- net ENC_A1: now also U$1.17/A3; no longer U$1.2
- net ENC_A2: now also U$1.14/A0; no longer U$1.4
- net ENC_B1: now also U$1.7; no longer U$1.1
- net ENC_B2: now also U$1.16/A2; no longer U$1.3
- net ENC_SW1: now also U$1.8; no longer U$1.0
- net ENC_SW2: now also U$1.15/A1; no longer U$1.21/A7
- net I1: now also JP1.5; no longer JP1.12
- net I2: now also JP2.5; no longer JP2.12, RI1.1
- net I3: now also JP8.5; no longer JP8.12, RI2.1
- net I4: now also JP11.5; no longer JP11.12, RI3.1
- net LIMA1: now also JP1.4; no longer JP1.5
- net LIMA2: now also JP2.4; no longer JP2.5
- net LIMA3: now also JP8.4; no longer JP8.5
- net LIMA4: now also JP11.4; no longer JP11.5
- net LIMB1: now also JP1.6; no longer JP1.7
- net LIMB2: now also JP2.6; no longer JP2.7
- net LIMB3: now also JP8.6; no longer JP8.7
- net LIMB4: now also JP11.6; no longer JP11.7
- net MOSI_B: now also U$1.0; no longer U$1.23/A9
- net N$35: now also JP2.8; no longer JP2.6
- net N$50: now also JP8.8; no longer JP8.6
- net N$65: now also JP11.8; no longer JP11.6
- net P1: now also JP1.1; no longer JP1.9
- net P2: now also JP2.1; no longer JP2.9, RP1.2
- net P3: now also JP8.1; no longer JP8.9, RP2.2
- net P4: now also JP11.1; no longer JP11.9, RP3.2
- net RST_LCD: now also U$1.9; no longer U$1.7
- net RS_LCD: now also U$1.10; no longer U$1.6
- net SCK_B: now also U$1.1; no longer U$1.22/A8
- net VDD: now also JP1.11, JP1.2, JP11.11, JP11.2, JP2.11, JP2.2, JP8.11, JP8.2; no longer JP1.1, JP11.1, JP2.1, JP8.1
- net VMON1: now also JP1.7; no longer JP1.8
- net VMON2: now also JP2.7; no longer JP2.8
- net VMON2_B: now also U$1.22/A8; no longer U$1.19/A5
- net VMON3: now also JP8.7; no longer JP8.8
- net VMON3_B: now also U$1.20/A6; no longer U$1.17/A3
- net VMON4: now also JP11.7; no longer JP11.8
- net VMON4_B: now also U$1.18/A4; no longer U$1.15/A1
- net VSET1: now also JP1.10; no longer JP1.3
- net VSET2: now also JP2.10; no longer JP2.3
- net VSET3: now also JP8.10; no longer JP8.3
- net VSET4: now also JP11.10; no longer JP11.3
Routing:
- net VDD: track 0.00 -> 642.7 mm, vias 0 -> 13
- net 2.5V: track 0.00 -> 300.6 mm, vias 0 -> 1
- net DGND: track 0.00 -> 287.3 mm, vias 0 -> 4
- net CS_POT4: track 0.00 -> 265.6 mm, vias 0 -> 1
- net VMON4: track 0.00 -> 265.2 mm, vias 0 -> 2
- net SCK_B: track 0.00 -> 256.1 mm, vias 0 -> 4
- net MOSI_B: track 0.00 -> 253.8 mm, vias 0 -> 5
- net ACT_T4: track 0.00 -> 242.2 mm, vias 0 -> 2
- net VSET4: track 0.00 -> 198.0 mm
- net VMON3: track 0.00 -> 195.8 mm, vias 0 -> 2
- net CS_POT3: track 0.00 -> 190.3 mm, vias 0 -> 1
- net ACT_T3: track 0.00 -> 171.8 mm, vias 0 -> 2
- net VMON2: track 0.00 -> 166.5 mm, vias 0 -> 6
- net VSET2: track 0.00 -> 158.6 mm, vias 0 -> 2
- net VSET3: track 0.00 -> 152.0 mm
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- added copper zone on layer 1, net DGND
- added copper zone on layer 16, net DGND
Other:
- board text added: "+5V"
- board text added: "GND"

Commit message: Finished routing board
Still to do: review layout, add vias, clean up silkscreen
Parts:
- added U$2: (no value), JQI_Logo:JQI_LOGO_NEGATIVE-SILKSCREEN
- moved R89 52.3 mm to (264.2, 20.3), turned to 180 degrees
- moved R71 50.7 mm to (191.1, 22.2)
- moved R53 50.2 mm to (118.1, 21.6)
- moved C22 18.8 mm to (210.2, 55.9)
- moved C23 18.5 mm to (210.2, 54.0)
- moved TP20 11.4 mm to (242.6, 64.8)
- moved C24 5.99 mm to (276.9, 55.2)
- moved C25 5.99 mm to (276.9, 53.3)
- moved IC10 5.68 mm to (283.2, 55.9)
- moved IC8 5.68 mm to (215.9, 55.9)
- moved TP25 5.24 mm to (289.6, 63.5)
- moved TP26 5.08 mm to (308.6, 64.8)
- moved TP19 2.84 mm to (221.0, 63.5)
- moved TP14 1.91 mm to (168.3, 64.8)
- moved TP24 1.80 mm to (283.2, 63.5)
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Routing:
- net VDD: track 642.7 -> 896.2 mm, vias 13 -> 21
- net VSET4: track 198.0 -> 299.3 mm, vias 0 -> 2
- net N$50: track 0.00 -> 85.9 mm, vias 0 -> 2
- net N$65: track 0.00 -> 80.6 mm, vias 0 -> 2
- net LIMB3: track 0.00 -> 78.4 mm, vias 0 -> 2
- net VSET3: track 152.0 -> 229.5 mm, vias 0 -> 2
- net LIMB4: track 0.00 -> 70.5 mm, vias 0 -> 2
- net VMON3: track 195.8 -> 262.6 mm, vias 2 -> 6
- net VMON4: track 265.2 -> 328.4 mm, vias 2 -> 4
- net ACT_T2: track 135.4 -> 82.4 mm
- net LIMA4: track 0.00 -> 49.6 mm, vias 0 -> 2
- net LIMA3: track 0.00 -> 46.9 mm, vias 0 -> 2
- net N$58: track 0.00 -> 26.5 mm, vias 0 -> 2
- net N$43: track 0.00 -> 25.2 mm, vias 0 -> 2
- net +1V_4: track 0.00 -> 22.3 mm, vias 0 -> 2
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- added copper zone on layer 1, net AGND
- added copper zone on layer 2, net AGND
- added copper zone on layer 2, net DGND
Other:
- board text added: "Temp Controller v0.9 BR"

Commit message: Board/Schematic updates and tweaks
Incorporate suggestions from Neal and Alessandro
Parts:
- L2: device rlc-jqi:0603 -> rlc-jqi:0805
- R28, R33: device rlc-jqi:0603 -> jqi_passives:R_0603
- moved L3 12.7 mm to (56.5, 56.5)
- moved R33 2.54 mm to (11.4, 16.5)
- moved R28 2.01 mm to (31.1, 15.9), turned to 90 degrees
- moved L1 1.27 mm to (64.8, 54.6)
- moved C27 0.64 mm to (64.1, 49.5)
- moved C30 0.64 mm to (64.1, 51.4)
Connections:
- net ENC_A1: now also R28.P$1; no longer R28.1
- net ENC_A2: now also R33.P$1; no longer R33.1
- net VDD: now also R28.P$2, R33.P$2; no longer R28.2, R33.2
Routing:
- net VDD: track 896.2 -> 909.2 mm, vias 21 -> 23
- net AGND: track 1.27 -> 10.9 mm, vias 5 -> 38
- net ENC_A2: track 42.7 -> 40.2 mm
- net MOSI_B: track 250.7 -> 253.0 mm
- net SCK_B: track 252.1 -> 254.1 mm
- net CS_DAC: track 36.7 -> 38.5 mm
- net CS_POT3: track 184.9 -> 185.9 mm
- net CS_POT4: track 256.5 -> 257.6 mm
- net CS_POT2: track 114.0 -> 115.0 mm
- net CS_POT1: track 41.1 -> 42.1 mm
- net ENC_A1: track 42.1 -> 41.1 mm
- net N$24: track 6.61 -> 5.80 mm
Other:
- board text added: "Temp Controller v0.9 BJR"
- board text removed: "Temp Controller v0.9 BR"

Commit message: Board/Schematic Clean up-lcd.init tweak
Added encoder hold event to initialize LCD to try to get around bug
where LCD display goes blank. The bug appears to be from a loose solder
connection on first prototype
Parts:
- added TP27: TESTPT, Lin-Temp-Controller:1206TESTPAD
- moved U$2 64.8 mm to (320.0, 1.27)
- moved R20 4.58 mm to (33.0, 24.1)
- moved R21 3.81 mm to (33.0, 26.7), turned to 180 degrees
- moved C3 1.80 mm to (34.3, 31.8), turned to 90 degrees
Connections:
- net AGND: now also TP27.P$1
Routing:
- net VMON4_B: track 8.27 -> 12.5 mm
- net LIMB3: track 78.4 -> 75.0 mm
- net ENC_SW1: track 44.4 -> 46.7 mm
- net VMON4: track 328.4 -> 329.4 mm, vias 4 -> 6
- net ENC_A1: track 41.1 -> 41.6 mm
Other:
- board text added: "DAC VREF"
- board text added: "VSET1"
- board text added: "VSET2"
- board text added: "VSET3"
- board text added: "VSET4"

Commit message: Add DAC Vref Jumper/Silkscreen Cleanup
Parts:
- added JP14: (no value), pinhead:1X02
- moved R15 4.49 mm to (71.8, 73.7)
- moved R31 0.64 mm to (19.7, 10.2)
- moved R34 0.63 mm to (14.6, 11.4)
Connections:
- net 2.5V: now also JP14.2
- net N$1: now also JP14.1
Routing:
- net N$1: track 4.24 -> 30.8 mm, vias 0 -> 1
- net 2.5V: track 302.7 -> 308.4 mm
- net ACT_T1: track 60.5 -> 59.3 mm
- net N$16: track 3.48 -> 4.12 mm
- net N$69: track 87.2 -> 87.8 mm
Other:
- board text added: "1V"
- board text added: "2.5V"
- board text added: "Cool Disable"
- board text added: "Ext Vref"
- board text added: "Heat Disable"
- board text added: "I"
- board text added: "Max V"
- board text added: "Min V"
- board text added: "P"
- board text added: "Temp"
- board text added: "VSET Protection Circuit"
- board text added: "Voltage"

Commit message: Add BOM, minor updates to reflect part availability
Parts:
- removed LCD_HEADER1: 2x8Header, mcu-accessories:ML16
- added LCD_HEADER: (no value), mcu-accessories:ML08
- C1: value 10nF -> 0.1uF
- C12, C20, C22, C24, C27: value 100nF -> 0.1uF
- C13, C2, C21, C23, C25, C30: device rlc-jqi:0603 -> rlc-jqi:0805
- C15: value .1uF -> 0.1uF
- R20, R21, R22, R23, R24, R25, R26, R27: value 10k -> 10k 1%
- moved L2 0.63 mm to (57.8, 32.4)
- moved C30 0.25 mm to (63.9, 51.4)
- renumbered L5 to L4
Connections:
- net 3.3V: now also LCD_HEADER.1; no longer LCD_HEADER1.13
- net CS_LCD: now also LCD_HEADER.6; no longer LCD_HEADER1.5
- net DGND: now also LCD_HEADER.2, LCD_HEADER.4; no longer LCD_HEADER1.11
- net MOSI: now also LCD_HEADER.3; no longer LCD_HEADER1.9
- net RST_LCD: now also LCD_HEADER.8; no longer LCD_HEADER1.1
- net RS_LCD: now also LCD_HEADER.7; no longer LCD_HEADER1.3
- net SCK: now also LCD_HEADER.5; no longer LCD_HEADER1.7
Routing:
- net MOSI: track 23.5 -> 19.0 mm
- net 3.3V: track 19.4 -> 15.5 mm
- net SCK: track 19.4 -> 16.5 mm
- net RST_LCD: track 26.5 -> 28.1 mm
- net RS_LCD: track 22.4 -> 21.2 mm
- net N$1: track 30.8 -> 31.6 mm
- net CS_LCD: track 17.3 -> 18.0 mm
- net N$25: track 6.54 -> 7.16 mm
Other:
- board text added: "Temp Controller v1.0 BJR"
- board text removed: "Temp Controller v0.9 BJR"

Commit message: Prepare for ordering boards
Update BOM, minor changes to board to move header slightly, ensure
silkscreen is using vector fonts
Connections:
- removed net MON: U$1.A14
Routing:
- net DGND: vias 6 -> 20
- net AGND: vias 38 -> 113
