File: v1_0 (first prod run)/mainBoard_v1_0/LinTempCont_4ch_V1_0.brd (EAGLE design)
At the start: 330.2 x 76.2 mm, 196 parts, among them IC1 LM393D, IC10 AD5262, IC2 LM393D, IC3 AD5624R, IC4 AD5262, IC5 AD5262, IC7 LM393D, IC8 AD5262, IC9 LM393D, T1 MMBT3904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

Commit message: Finish version 1
Reorganize file structure. Package version 1 files nicely along with BOM
in order to get boards assembled
Parts:
- turned D1 to 270 degrees
- turned D2 to 270 degrees
- turned D3 to 270 degrees
- turned D4 to 270 degrees
- turned IC1 to 0 degrees
- turned IC2 to 0 degrees
- turned IC6 to 180 degrees
- turned IC7 to 0 degrees
- turned IC9 to 0 degrees
- turned T1 to 180 degrees
- turned T2 to 0 degrees
- turned T3 to 180 degrees
- turned T4 to 0 degrees
- turned T5 to 180 degrees
- turned T6 to 0 degrees
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